File: hardware/ubertooth-one/ubertooth-one.sch (KiCad schematic (older format))
At the start: 0 parts

Commit message: LPC175x symbol
Parts:
- added U?: LPC175X, symbol LPC175X
Changed lines of the file:
@@
-EESchema Schematic File Version 2  date Wed Nov  3 19:58:18 2010
+EESchema Schematic File Version 2  date Wed Nov  3 22:50:43 2010
+LIBS:ubertooth-symbols
 LIBS:power
 LIBS:device
@@
 LIBS:contrib
 LIBS:valves
-EELAYER 43  0
+LIBS:ubertooth-one-cache
+EELAYER 24  0
 EELAYER END
-$Descr A4 11700 8267
+$Descr User 17000 11000
 Sheet 1 1
 Title ""
@@
 Comment4 ""
 $EndDescr
+$Comp
+L LPC175X U?
+U 1 1 4CD23A14
+P 11400 5550
+F 0 "U?" H 11400 5650 60  0000 C CNN
+F 1 "LPC175X" H 11400 5450 60  0000 C CNN
+	1    11400 5550
+	0    -1   -1   0
+$EndComp
 $EndSCHEMATC

Commit message: CC2400, CC2591
Parts:
- added U?: CC2400, symbol CC2400
Changed lines of the file:
@@
-EESchema Schematic File Version 2  date Wed Nov  3 22:50:43 2010
+EESchema Schematic File Version 2  date Thu Nov  4 21:27:38 2010
 LIBS:ubertooth-symbols
 LIBS:power
@@
 $EndDescr
 $Comp
+L CC2400 U?
+U 1 1 4CD3795B
+P 6350 2900
+F 0 "U?" H 6350 3000 60  0000 C CNN
+F 1 "CC2400" H 6350 2800 60  0000 C CNN
+	1    6350 2900
+	1    0    0    -1
+$EndComp
+$Comp
 L LPC175X U?

Commit message: ubertooth one schematic
Parts:
- added C1, C4, C5: 68pF, symbol C
- added C101: 18pF, symbol C
- added C102, C12, C132, C161: 1nF, symbol C
- added C11, C131: 10pF, symbol C
- added C111: 1pF, symbol C
- added C112: 6p8, symbol C
- added C113: 2p2, symbol C
- added C14, C15, C16, C17, C18, C2, C20, C6, C7: 100nF, symbol C
- added C19, C21, C23, C24, C433, C435: 1µF, symbol C
- added C3, C432, C434: 10nF, symbol C
- added C421, C431: 27pF, symbol C
- added C8: 220pF, symbol C
- added C9: 100pF, symbol C
- added D1: 1V8LED, symbol LED
- added D2: TXLED, symbol LED
- added D3: RXLED, symbol LED
- added D4: USRLED, symbol LED
- added D5: RSTLED, symbol LED
- added D6: USBLED, symbol LED
- added FB1, FB2, FB3, FB4: FILTER, symbol FILTER
- added J1: USB-DEVICE, symbol USB-DEVICE
- added L111: 2n2, symbol INDUCTOR
- added L112: 3nH, symbol INDUCTOR
- added L21: DNP, symbol INDUCTOR
- added P1: SMA-CONN, symbol SMA-CONN
- added P2: PROGRAM, symbol CONN_6
- added P3: JTAG, symbol CONN_5X2
- added P4: EXPAND, symbol CONN_3X2
- added Q1: PMBT3906, symbol PNP
- added R1, R10, R13, R453: 10k, symbol R
- added R11, R5, R6, R7, R8, R9: 330, symbol R
- added R151: 4k3, symbol R
- added R2, R3: 33, symbol R
- added R4: 1k5, symbol R
- added R451: 43k, symbol R
- added R452: 2k2, symbol R
- added U3: BU33TA2, symbol BUXXTA2
- added U4: BU18TA2, symbol BUXXTA2
- added U5: IP4221CZ6, symbol IP4221CZ6
- added U6: CC2591, symbol CC2591
- added X1: ABMM2, symbol CRYSTAL
- gave numbers to parts that had none: 2
Connections:
- net at U2.1 (TDO/SWO): now also P3.6
- net VREFP: now reaches U2.10 (VREFP)
- net VREFP: now also C434.2, C435.2, FB3.1
- net at U2.11 (RSTOUT): now also R8.2
- net VREFN: now reaches U2.12 (VREFN)
- net VREFN: now also C434.1, C435.1, FB4.1
- net at U2.14 (RESET): now also P2.2, P3.10, R1.2
- net 3V3: now reaches U2.16 (VBAT)
- net 3V3: now also U2.21 (VDD(3V3)), U2.34 (VDD(REG)(3V3)), U2.42 (VDD(3V3)), U2.56 (VDD(3V3)), U2.67 (VDD(REG)(3V3)), U2.77 (VDD(3V3)), C101.2, C102.2, C11.1, C12.1, C131.1, C132.1, C14.1, C15.2, C16.1, C161.1, C17.2, C18.1, C20.1, C21.2, D6.1 (A), FB1.2, FB3.2, P3.1, Q1.1 (E), R1.1, R13.2, R453.2, U3.1 (VOUT), U6.1 (AVDD_PA1), U6.10 (AVDD_PA2), U6.13 (AVDD_LNA), U6.16 (AVDD_BIAS)
- net VBUS: now reaches U2.18 (P1[30]/VBUS/AD0[4])
- net VBUS: now also C19.2, C23.2, J1.1 (VBUS), U3.3 (STBY), U3.4 (VIN), U4.4 (VIN), U5.5 (VCC)
- net at U2.19 (XTAL1): now also C8.1, C9.2
- net at U2.2 (TDI): now also P3.8
- net at U2.22 (P0[29]/USB_D+): now also R2.2
- net at U2.23 (P0[30]/USB_D-): now also R3.2
- net GND: now reaches U2.24 (VSS)
- net GND: now also U1.18 (DGND_GUARD), U1.22 (DGND), U1.23 (DSUB_PADS), U1.24 (DSUB_CORE), U1.49 (AGND), U1.5 (GND), U1.9 (GND), U2.33 (VSS), U2.43 (VSS), U2.57 (VSS), U2.66 (VSS), U2.78 (VSS), C1.2, C101.1, C102.1, C11.2, C111.1, C113.1, C12.2, C131.2, C132.2, C14.2, C15.1, C16.2, C161.2, C17.1, C18.2, C19.1, C2.2, C20.2, C21.1, C23.1, C24.2, C3.2, C4.2, C421.2, C431.2, C5.1, C6.1, C7.1, C8.2, D1.2 (K), D2.2 (K), D3.2 (K), D4.2 (K), D5.2 (K), FB2.2, FB4.2, J1.4 (GND), L112.1, P1.2 (GND), P1.3 (GND), P1.4 (GND), P1.5 (GND), P2.1, P3.3, P3.5, P3.9, P4.1, R10.1, R151.2, R451.1, U3.2 (GND), U4.2 (GND), U5.2 (GND), U6.12 (GND), U6.14 (GND), U6.17 (GND), U6.8 (GND), U6.9 (GND)
- net at U2.25 (P1[18]/USB_UP_LED/PWM1[1]/CAP1[0]): now also R5.2
- net at U2.3 (TMS/SWDIO): now also P3.2
- net ISP: now reaches U2.41 (P2[10]/EINT0/NMI)
- net ISP: now also P2.6, R13.1
- net at U2.45 (P0[18]/DCD1/MOSI0/MOSI): now also P4.2
- net at U2.46 (P0[17]/CTS1/MISO0/MISO): now also P4.4
- net at U2.47 (P0[15]/TXD1/SCK0/SCK): now also P4.6
- net at U2.48 (P0[16]/RXD1/SSEL0/SSEL): now also P4.5
- net USB_CONNECT: now reaches U2.49 (P2[9]/USB_CONNECT/RXD2)
- net USB_CONNECT: now also R452.2
- net at U2.5 (TCK/SWDCLK): now also P3.4
- net at U2.50 (P2[8]/TD2/TXD2): now also U6.7 (HGM)
- net at U2.51 (P2[7]/RD2/RTS1): now also U6.6 (EN)
- net at U2.52 (P2[6]/PCAP1[0]/RI1/TRACECLK): now also U6.5 (PAEN)
- net at U2.53 (P2[5]/PWM1[6]/DTR1/TRACEDATA[0]): now also U1.35 (GIO6)
- net at U2.54 (P2[4]/PWM1[5]/DSR1/TRACEDATA[1]): now also U1.34 (SO)
- net at U2.58 (P2[2]/PWM1[3]/CTS1/TRACEDATA[3]): now also U1.33 (SI)
- net at U2.59 (P2[1]/PWM1[2]/RXD1): now also U1.32 (SCLK)
- net ATEST2: now reaches U2.6 (P0[26]/AD0[3]/AOUT/RXD3)
- net ATEST2: now also U1.46 (ATEST2)
- net at U2.60 (P2[0]/PWM1[1]/TXD1): now also U1.31 (CSn)
- net at U2.61 (P0[9]/I2STX_SDA/MOSI1/MAT2[3]): now also U1.29 (DIO/PKT), U2.62 (P0[8]/I2STX_WS/MISO1/MAT2[2])
- net at U2.63 (P0[7]/I2STX_CLK/SCK1/MAT2[1]): now also U1.30 (DCLK/FIFO)
- net at U2.64 (P0[6]/I2SRX_SDA/SSEL1/MAT2[0]): now also U2.65 (P4[28]/RX_MCLK/MAT2[0]/TXD3)
- net at U2.68 (P4[29]/TX_MCLK/MAT2[1]/RXD3): now also U1.28 (TX)
- net at U2.69 (P1[15]/ENET_REF_CLK): now also U1.27 (RX)
- net ATEST1: now reaches U2.7 (P0[25]/AD0[2]/I2SRX_SDA/TXD3)
- net ATEST1: now also U1.47 (ATEST1)
- net at U2.70 (P1[14]/ENET_RX_ER): now also U1.25 (DVDD3.3), C7.2
- net at U2.71 (P1[10]/ENET_RXD1): now also U1.20 (BT/GR)
- net at U2.72 (P1[9]/ENET_RXD0): now also R10.2, R11.2, U4.3 (STBY)
- net at U2.73 (P1[8]/ENET_CRS): now also R7.2
- net at U2.74 (P1[4]/ENET_TX_EN): now also R6.2
- net at U2.75 (P1[1]/ENET_TXD1): now also R9.2
- net at U2.79 (P0[2]/TXD0/AD0[7]): now also P2.5
- net VDDA: now reaches U2.8 (VDDA)
- net VDDA: now also C432.2, C433.2, FB1.1
- net at U2.80 (P0[3]/RXD0/AD0[6]): now also P2.4
- net VSSA: now reaches U2.9 (VSSA)
- net VSSA: now also C432.1, C433.1, FB2.1
- net +1.8V: now reaches U1.1 (VCO_GUARD)
- net +1.8V: now also U1.10 (AVDD_SW), U1.14 (AVDD_RF2), U1.15 (AVDD_IF2), U1.16 (AVDD_ADC), U1.17 (DVDD_ADC), U1.19 (GUARD), U1.2 (AVDD_VCO), U1.26 (DVDD1.8), U1.3 (AVDD_PRE), U1.4 (AVDD_RF1), U1.41 (AVDD_XOSC), U1.44 (AVDD_IF1), U1.48 (AVDD_CHP), C1.1, C2.1, C24.1, C3.1, C4.1, C5.2, C6.2, U4.1 (VOUT)
- net GIO1: now reaches U1.21 (GIO1)
- net GIO1: now also C9.1
- net at U1.42 (XOSC16_Q2): now also C421.1, X1.2
- net at U1.43 (XOSC16_Q1): now also C431.1, X1.1
- net at U1.45 (R_BIAS): now also R451.2
- net at U1.6 (RF_P): now also L21.1, U6.4 (RF_P)
- net at U1.7 (TXRX_SWITCH): now also U6.3 (TXRX)
- net at U1.8 (RF_N): now also L21.2, U6.2 (RF_N)
- new net: C112.1, U6.11 (ANT)
- new net: R151.1, U6.15 (BIAS)
- new net: J1.3 (D+), R2.1, R4.2, U5.4 (ESD3)
- new net: J1.2 (D-), R3.1, U5.6 (ESD4)
- new net: Q1.3 (C), R4.1
- new net: Q1.2 (B), R452.1, R453.1
- new net: D5.1 (A), R8.1
- new net: D6.2 (K), R5.1
- new net: D4.1 (A), R9.1
- new net: D3.1 (A), R6.1
- new net: D2.1 (A), R7.1
- new net: D1.1 (A), R11.1
- new net: C111.2, C112.2, L111.2
- new net: C113.2, L111.1, L112.2, P1.1 (RF)
- no-connect marks 0 -> 34
Other:
- note added: "JTAG connector"
- note added: "expansion\nconnector"
- note added: "optional ADC section"
- note added: "programming\n connector"
- note added: "transmission\nline inductor"
- moved on the sheet: U1, U2
