File: hardware/ubertooth-one/ubertooth-one.sch (KiCad schematic (older format))
At the start: 77 parts, among them J1 USB-DEVICE, P1 SMA-CONN, P2 PROGRAM, P3 JTAG, P4 EXPAND, Q1 PMBT3906, U1 CC2400, U2 LPC175X, U3 BU33TA2, U4 BU18TA2, U5 IP4221CZ6, U6 CC2591, X1 ABMM2

Commit message: ubertooth one layout complete this is an attempt at a two layer board - it will probably turn into four layers
Parts:
- renumbered C113 to C1, C434 to C10, C435 to C11, C161 to C12, C11 to C13, C12 to C14, C1 to C15, C2 to C16, C3 to C17, C24 to C18, C431 to C19, C102 to C2, C5 to C20, C421 to C21, C23 to C22, C4 to C23, C6 to C24, C7 to C25, C15 to C26, C14 to C27, C16 to C28, C8 to C29, C111 to C3, C17 to C30, C9 to C31, C21 to C32, C20 to C33, C18 to C34, C19 to C35, C101 to C4, C112 to C5, C132 to C6, C432 to C7, C433 to C8, C131 to C9, L112 to L1, L111 to L2, L21 to L3, R151 to R1, R13 to R10, R452 to R11, R3 to R12, R2 to R13, R453 to R14, R5 to R15, R4 to R16, R451 to R2, R10 to R3, R11 to R4, R7 to R5, R9 to R7, R1 to R9, U6 to U1, U4 to U2, U1 to U3, U2 to U4, U3 to U5, U5 to U6
Connections:
- net VDDA is gone; now on net 3V3: C7.2, C8.2, FB1.1, U4.8 (VDDA)
- net VREFN is gone; now on net GND: C10.1, C11.1, FB4.1, U4.12 (VREFN)
- net VREFP is gone; now on net 3V3: C10.2, C11.2, FB3.1, U4.10 (VREFP)
- net VSSA is gone; now on net GND: C7.1, C8.1, FB2.1, U4.9 (VSSA)
- net GND: now also U2.0, U5.0
- net at U4.45 (P0[18]/DCD1/MOSI0/MOSI): now also P4.6; no longer P4.2
- net at U4.47 (P0[15]/TXD1/SCK0/SCK): now also P4.2; no longer P4.6
- net at U4.53 (P2[5]/PWM1[6]/DTR1/TRACEDATA[0]): now also U3.31 (CSn); no longer U3.35 (GIO6)
- net at U4.54 (P2[4]/PWM1[5]/DSR1/TRACEDATA[1]): now also U3.32 (SCLK); no longer U3.34 (SO)
- net at U4.58 (P2[2]/PWM1[3]/CTS1/TRACEDATA[3]): now also U3.35 (GIO6); no longer U3.33 (SI)
- net at U4.59 (P2[1]/PWM1[2]/RXD1): now also U3.34 (SO); no longer U3.32 (SCLK)
- net at U4.60 (P2[0]/PWM1[1]/TXD1): now also U3.33 (SI); no longer U3.31 (CSn)
Other:
- moved on the sheet: P4

Commit message: ubertooth one tweaks
Parts:
- added R17, R18: 0, symbol R
Connections:
- net 3V3: now also R17.1
- net VBUS: now also R18.1
- net at U4.44 (P0[22]/RTS1/TD1): now also P4.3
- net at P2.3: now also R17.2, R18.2
- no-connect marks 34 -> 31
Other:
- note added: "DNP"

Commit message: filling in some bill of materials information
Parts:
- C1: footprint (none) -> SM0402; Field1 (none) -> Murata; Field2 (none) -> GRM1555C1H2R2BZ01D; Field3 (none) -> Multilayer Ceramic Capacitors (MLCC) - SMD/SMT 0402 2.2pF 5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
- C10, C11, C15, C16, C17, C18, C19, C20, C21, C22, C23, C24, C25, C26, C27, C28, C29, C30, C31, C32, C33, C34, C35, C7, C8, L3, R1, R10, R11, R12, R13, R14, R15, R16, R2, R3, R4, R5, R6, R7, R8, R9: footprint (none) -> SM0402
- C12, C14, C6: footprint (none) -> SM0402; Field1 (none) -> Murata; Field2 (none) -> GRM1555C1H102JA01D
- C13, C9: footprint (none) -> SM0402; Field1 (none) -> Murata; Field2 (none) -> GRM1555C1H100JZ01D; Field3 (none) -> Multilayer Ceramic Capacitors (MLCC) - SMD/SMT 0402 10pF 50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
- C2: footprint (none) -> SM0402; Field1 (none) -> Murata; Field2 (none) -> GRM1555C1H102JA01D; Field3 (none) -> Multilayer Ceramic Capacitors (MLCC) - SMD/SMT 0402 1000pF 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
- C3: footprint (none) -> SM0402; Field1 (none) -> Murata; Field2 (none) -> GRM1555C1H1R0BZ01D; Field3 (none) -> Multilayer Ceramic Capacitors (MLCC) - SMD/SMT 0402 1.0pF 5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
- C4: footprint (none) -> SM0402; Field1 (none) -> Murata; Field2 (none) -> GRM1555C1H180JZ01J; Field3 (none) -> Multilayer Ceramic Capacitors (MLCC) - SMD/SMT 0402 18pF 50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
- C5: footprint (none) -> SM0402; Field1 (none) -> Murata; Field2 (none) -> GRM1555C1H6R8BZ01D; Field3 (none) -> Multilayer Ceramic Capacitors (MLCC) - SMD/SMT 0402 6.8pF 5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
- D1, D2, D3, D4, D5, D6: footprint (none) -> LED-0603
- FB1, FB2, FB3, FB4, R17, R18: footprint (none) -> SM0603
- J1: footprint (none) -> USB-A-MOLEX-480371000
- L1: footprint (none) -> SM0402; Field1 (none) -> Murata; Field2 (none) -> LQG15HN3N0S02D; Field3 (none) -> RF Inductor
- L2: footprint (none) -> SM0402; Field1 (none) -> Murata; Field2 (none) -> LQG15HS2N2S02D; Field3 (none) -> RF Inductor
- P1: footprint (none) -> SMA-EDGE
- P2: footprint (none) -> 100MIL-HEADER-1X6-EDGE
- P3: footprint (none) -> 50MIL-HEADER-2X5-TH
- P4: footprint (none) -> PIN_ARRAY_3X2
- Q1: footprint (none) -> SOT883
- U1: footprint (none) -> VQFN16
- U2, U5: footprint (none) -> SSON004X1216
- U3: footprint (none) -> QFN48
- U4: footprint (none) -> LQFP80
- U6: footprint (none) -> SOT886
- X1: footprint (none) -> ABMM2

Commit message: finished bill of materials info
Parts:
- C15, C20, C23: Field1 (none) -> Murata; Field2 (none) -> GRM1555C1H680JZ01D; Field3 (none) -> Multilayer Ceramic Capacitors (MLCC) - SMD/SMT 68PF 50V 5%
- C16, C24, C25, C26, C27, C28, C30, C33, C34: Field1 (none) -> Murata; Field2 (none) -> GRM155R71C104KA88D; Field3 (none) -> Multilayer Ceramic Capacitors (MLCC) - SMD/SMT 0402 0.1uF 1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
- C17: Field1 (none) -> Murata; Field2 (none) -> GRM155R71E103KA01D; Field3 (none) -> Multilayer Ceramic Capacitors (MLCC) - SMD/SMT 0402 0.01uF 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
- C18, C22, C32, C35: Field1 (none) -> TDK; Field2 (none) -> C1005X5R1C105K; Field3 (none) -> Multilayer Ceramic Capacitors (MLCC) - SMD/SMT 0402 1.0uF 1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
- C19, C21: Field1 (none) -> Murata; Field2 (none) -> GRM1555C1H270JZ01J; Field3 (none) -> Multilayer Ceramic Capacitors (MLCC) - SMD/SMT 27pF 50 volt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
- C29: Field1 (none) -> Murata; Field2 (none) -> GRM1555C1E221JA01D; Field3 (none) -> Multilayer Ceramic Capacitors (MLCC) - SMD/SMT 0402 220pF 2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
- C31: Field1 (none) -> Murata; Field2 (none) -> GRM1555C1H101JZ01D; Field3 (none) -> Multilayer Ceramic Capacitors (MLCC) - SMD/SMT 0402 100pF 5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
- D1, D5: Field1 (none) -> Kingbright; Field2 (none) -> APT1608SGC; Field3 (none) -> Standard LED - SMD GREEN WATER CLEAR
- D2: Field1 (none) -> OSRAM; Field2 (none) -> LY L29K-H1K2-26-Z; Field3 (none) -> Standard LED - SMD Yellow, 587nm 28mcd, 2mA
- D3: Field1 (none) -> OSRAM; Field2 (none) -> LO L29K-J2L1-24-Z; Field3 (none) -> Standard LED - SMD Orange, 606nm 14mcd, 2mA
- D4, D6: Field1 (none) -> Kingbright; Field2 (none) -> APT1608EC; Field3 (none) -> Standard LED - SMD HI EFF RED WTR CLR
- J1: Field1 (none) -> Molex; Field2 (none) -> 48037-1000; Field3 (none) -> USB & Firewire Connectors TYPE A RA SHLDED PLG SMT AU
- Q1: Field1 (none) -> NXP; Field2 (none) -> PMBT3906M,315; Field3 (none) -> Bipolar Small Signal GENERAL PURPOSE TRANSISTOR
- R1: Field1 (none) -> KOA Speer; Field2 (none) -> RK73H1ETTP4301F; Field3 (none) -> Thick Film Resistors - SMD 1/16watt 4.3Kohms 1%
- R10, R14, R3, R9: Field1 (none) -> Vishay/Dale; Field2 (none) -> CRCW040210K0JNED; Field3 (none) -> Thick Film Resistors - SMD 1/16watt 10Kohms 5%
- R11: Field1 (none) -> Vishay/Dale; Field2 (none) -> CRCW04022K20JNED; Field3 (none) -> Thick Film Resistors - SMD 1/16watt 2.2Kohms 5%
- R12, R13: Field1 (none) -> Vishay/Dale; Field2 (none) -> CRCW040233R0FKED; Field3 (none) -> Thick Film Resistors - SMD 1/16watt 33ohms 1% 100ppm
- R15, R4, R5, R6, R7, R8: Field1 (none) -> Vishay/Dale; Field2 (none) -> CRCW0402330RJNED; Field3 (none) -> Thick Film Resistors - SMD 1/16watt 330ohms 5%
- R16: Field1 (none) -> Vishay/Dale; Field2 (none) -> CRCW04021K50JNED; Field3 (none) -> Thick Film Resistors - SMD 1/16watt 1.5Kohms 5%
- R2: Field1 (none) -> KOA Speer; Field2 (none) -> RK73H1ETTP4302F; Field3 (none) -> Thick Film Resistors - SMD 1/16watts 43Kohms 1%
- U1: Field1 (none) -> Texas Instruments; Field2 (none) -> CC2591RGVR; Field3 (none) -> RF Front End 2.4 GHz
- U2: Field1 (none) -> ROHM; Field2 (none) -> BU18TA2WNVX-TR; Field3 (none) -> Low Dropout (LDO) Regulators High-Speed Load CMOS 1.8V Out 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
- U3: Field1 (none) -> Texas Instruments; Field2 (none) -> CC2400-RTB1; Field3 (none) -> RF Receiver Lo-Pwr Sgl-Chip 2.4 GHz ISM Band Trnscvr
- U4: Field1 (none) -> NXP; Field2 (none) -> LPC1758FBD80,551; Field3 (none) -> Microcontrollers (MCU) ARM Cortex M3 Micro Controller
- U5: Field1 (none) -> ROHM; Field2 (none) -> BU33TA2WNVX-TR; Field3 (none) -> Low Dropout (LDO) Regulators High-Speed Load CMOS 3.3V Out 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
- U6: Field1 (none) -> NXP; Field2 (none) -> IP4221CZ6-XS,132; Field3 (none) -> ESD Suppressors Dual USB 2.0 Integra ESD Protection 6-Pin
- X1: Field1 (none) -> Abracon; Field2 (none) -> ABMM2-16.000MHZ-E2-T; Field3 (none) -> Crystals +/-20PPM 16MHz

Commit message: updated 2 layer programming pinout
Parts:
- removed R17, R18: 0, SM0603, symbol R
Connections:
- net ISP: now also P2.2; no longer P2.6
- net at P3.10, R9.2, U4.14 (RESET): now also P2.6; no longer P2.2
- no-connect marks 31 -> 32
Other:
- note removed: "DNP"
- moved on the sheet: P2

Commit message: merged 4layer branch to trunk
Parts:
- removed C13: 10pF, SM0402, symbol C
- removed Q1: PMBT3906, SOT883, symbol PNP
- removed U2: BU18TA2, SSON004X1216, symbol BUXXTA2
- removed U5: BU33TA2, SSON004X1216, symbol BUXXTA2
- removed U6: IP4221CZ6, SOT886, symbol IP4221CZ6
- added C36: 15pF, 0402, symbol C
- added P10: ATEST1, symbol CONN_1
- added P11: ATEST2, symbol CONN_1
- added P12: DCLK, symbol CONN_1
- added P13: DIO, symbol CONN_1
- added P5: 1V8, symbol CONN_1
- added P6: 3V3, symbol CONN_1
- added P7: VBUS, symbol CONN_1
- added P8: GIO1, symbol CONN_1
- added P9: GIO6, symbol CONN_1
- added Q1: BC856, SOT416, symbol BC856
- added R17: 10k, 0603, symbol R
- added R18: 49.9k, 0402, symbol R
- added R19: 30.1k, 0402, symbol R
- added U6: IP4220CZ6, SOT457, symbol IP4220CZ6
- added U7: TPS71219, S-PVSON-N10, symbol TPS712XX
- C1, C16, C17, C2, C24, C25, C3, C4, C9, L1: footprint SM0402 -> 0402
- C10, C11, C7, C8: footprint SM0402 -> 0603
- C12, C14, C6: footprint SM0402 -> 0402; Field3 (none) -> Multilayer Ceramic Capacitors (MLCC) - SMD/SMT 0402 1000pF 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
- C15, C20, C23: footprint SM0402 -> 0402; Field3 Multilayer Ceramic Capacitors (MLCC) - SMD/SMT 68PF 50V 5% -> Multilayer Ceramic Capacitors (MLCC) - SMD/SMT 0402 68PF 50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
- C18, C32: value 1µF -> 2.2µF; footprint SM0402 -> 0603; Field2 C1005X5R1C105K -> C1608X5R1C225K; Field3 Multilayer Ceramic Capacitors (MLCC) - SMD/SMT 0402 1.0uF 1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 -> Multilayer Ceramic Capacitors (MLCC) - SMD/SMT 0603 16volts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
- C19, C21: footprint SM0402 -> 0402; Field1 Murata -> TDK; Field2 GRM1555C1H270JZ01J -> C1608C0G1H270J; Field3 Multilayer Ceramic Capacitors (MLCC) - SMD/SMT 27pF 50 volt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 -> Multilayer Ceramic Capacitors (MLCC) - SMD/SMT 0603 27pF 50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
- C22: footprint SM0402 -> 0603; Field2 C1005X5R1C105K -> C1608X5R1C105K; Field3 Multilayer Ceramic Capacitors (MLCC) - SMD/SMT 0402 1.0uF 1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 -> Multilayer Ceramic Capacitors (MLCC) - SMD/SMT 0603 1uF 16v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
- C26, C27, C28, C30, C33, C34: footprint SM0402 -> 0603; Field1 Murata -> TDK; Field2 GRM155R71C104KA88D -> C1608X7R1H104K; Field3 Multilayer Ceramic Capacitors (MLCC) - SMD/SMT 0402 0.1uF 1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 -> Multilayer Ceramic Capacitors (MLCC) - SMD/SMT 0603 0.1uF 5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
- C29: footprint SM0402 -> 0603; Field1 Murata -> TDK; Field2 GRM1555C1E221JA01D -> C1608X7R1H221K; Field3 Multilayer Ceramic Capacitors (MLCC) - SMD/SMT 0402 220pF 2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 -> Multilayer Ceramic Capacitors (MLCC) - SMD/SMT 0603 220pF 5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
- C31: footprint SM0402 -> 0603; Field1 Murata -> TDK; Field2 GRM1555C1H101JZ01D -> C1608C0G1H101J; Field3 Multilayer Ceramic Capacitors (MLCC) - SMD/SMT 0402 100pF 5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 -> Multilayer Ceramic Capacitors (MLCC) - SMD/SMT 0603 100pF 5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
- C35: value 1µF -> 10nF; footprint SM0402 -> 0402; Field1 TDK -> Murata; Field2 C1005X5R1C105K -> GRM155R71E103KA01D; Field3 Multilayer Ceramic Capacitors (MLCC) - SMD/SMT 0402 1.0uF 1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 -> Multilayer Ceramic Capacitors (MLCC) - SMD/SMT 0402 0.01uF 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
- C5: footprint SM0402 -> 0402; Field2 GRM1555C1H6R8BZ01D -> GRM1555C1H6R8CZ01D
- D1, D2, D3, D4, D5, D6: footprint LED-0603 -> 0603D
- FB1, FB2, FB3, FB4: footprint SM0603 -> 0603bridged
- L2: footprint SM0402 -> 0402; Field2 LQG15HS2N2S02D -> LQW15AN2N2C10D; Field3 RF Inductor -> Power Inductors 2.2 NH +-.2NH
- L3: footprint SM0402 -> 0402gap
- P1: Field1 (none) -> Connector City; Field2 (none) -> CONREVSMA003.062; Field3 (none) -> RF Connectors RP-SMA Fml Edge Mnt for 0.062 Thick Brd
- R1: footprint SM0402 -> 0402; Field3 Thick Film Resistors - SMD 1/16watt 4.3Kohms 1% -> Thick Film Resistors - SMD 0402 1/16watt 4.3Kohms 1%
- R10, R14, R3, R9: footprint SM0402 -> 0603; Field1 Vishay/Dale -> Bourns; Field2 CRCW040210K0JNED -> CR0603-JW-103ELF; Field3 Thick Film Resistors - SMD 1/16watt 10Kohms 5% -> Thick Film Resistors - SMD 0603 10KOHMS 5% 1/10WATT
- R11: footprint SM0402 -> 0603; Field1 Vishay/Dale -> Bourns; Field2 CRCW04022K20JNED -> CR0603-JW-222ELF; Field3 Thick Film Resistors - SMD 1/16watt 2.2Kohms 5% -> Thick Film Resistors - SMD 0603 2.2KOHMS 5% 1/10WATT
- R12, R13: footprint SM0402 -> 0603; Field2 CRCW040233R0FKED -> CRCW060333R0FKEA; Field3 Thick Film Resistors - SMD 1/16watt 33ohms 1% 100ppm -> Thick Film Resistors - SMD 0603 1/16watt 33ohms 1% 100ppm
- R15, R4, R5, R6, R7, R8: footprint SM0402 -> 0603; Field1 Vishay/Dale -> Bourns; Field2 CRCW0402330RJNED -> CR0603-JW-331ELF; Field3 Thick Film Resistors - SMD 1/16watt 330ohms 5% -> Thick Film Resistors - SMD 0603 330OHMS 5% 1/10WATT
- R16: footprint SM0402 -> 0603; Field1 Vishay/Dale -> Bourns; Field2 CRCW04021K50JNED -> CR0603-JW-152ELF; Field3 Thick Film Resistors - SMD 1/16watt 1.5Kohms 5% -> Thick Film Resistors - SMD 0603 1.5KOHMS 5% 1/10WATT
- R2: footprint SM0402 -> 0402; Field3 Thick Film Resistors - SMD 1/16watts 43Kohms 1% -> Thick Film Resistors - SMD 0402 1/16watts 43Kohms 1%
- U4: Field2 LPC1758FBD80,551 -> LPC1754FBD80,551
Connections:
- net +1.8V: now also P5.1, U7.3 (OUT1)
- net 3V3: now also C32.1, C36.1, P6.1, Q1.2 (E), R18.1, U7.4 (OUT2); no longer C10.2, C11.2, C32.2, C7.2, C8.2, FB1.1, FB3.1, U4.10 (VREFP), U4.8 (VDDA)
- net ATEST1: now also P10.1
- net ATEST2: now also P11.1
- net GIO1: now also P8.1
- net GND: now also C22.2, C32.2, C35.2, R17.2, R19.2, U6.2 (GND), U7.0, U7.5 (GND); no longer C10.1, C11.1, C22.1, C32.1, C35.1, C7.1, C8.1, FB2.1, FB4.1, U4.12 (VREFN), U4.9 (VSSA)
- net VBUS: now also C22.1, P7.1, U6.5 (VP), U7.1 (IN), U7.8 (EN2); no longer C22.2, C35.2
- net HGM: now reaches U1.7 (HGM), U4.50 (P2[8]/TD2/TXD2)
- net EN: now reaches U1.6 (EN), U4.51 (P2[7]/RD2/RTS1)
- net EN: now also U1.5 (PAEN), R17.1
- net at U4.52 (P2[6]/PCAP1[0]/RI1/TRACECLK): no longer U1.5 (PAEN)
- net CSn: now reaches U3.31 (CSn), U4.53 (P2[5]/PWM1[6]/DTR1/TRACEDATA[0])
- net SCLK: now reaches U3.32 (SCLK), U4.54 (P2[4]/PWM1[5]/DSR1/TRACEDATA[1])
- net GIO6: now reaches U3.35 (GIO6), U4.58 (P2[2]/PWM1[3]/CTS1/TRACEDATA[3])
- net GIO6: now also P9.1
- net SO: now reaches U3.34 (SO), U4.59 (P2[1]/PWM1[2]/RXD1)
- net SI: now reaches U3.33 (SI), U4.60 (P2[0]/PWM1[1]/TXD1)
- net DIO: now reaches U3.29 (DIO/PKT), U4.61 (P0[9]/I2STX_SDA/MOSI1/MAT2[3]), U4.62 (P0[8]/I2STX_WS/MISO1/MAT2[2])
- net DIO: now also P13.1
- net DCLK: now reaches U3.30 (DCLK/FIFO), U4.63 (P0[7]/I2STX_CLK/SCK1/MAT2[1])
- net DCLK: now also P12.1
- net TX: now reaches U3.28 (TX), U4.68 (P4[29]/TX_MCLK/MAT2[1]/RXD3)
- net RX: now reaches U3.27 (RX), U4.69 (P1[15]/ENET_REF_CLK)
- net at R3.2, R4.2, U4.72 (P1[9]/ENET_RXD0): now also U7.10 (EN1)
- net at J1.3 (D+), R13.1, R16.2: now also U6.4 (ESD3)
- net at J1.2 (D-), R12.1: now also U6.6 (ESD4)
- net at R16.1: now also Q1.3 (C)
- net at R11.1, R14.1: now also Q1.1 (B)
- new net: C35.1, U7.6 (NR)
- new net: C36.2, R18.2, R19.1, U7.7 (FB2/NC)
- new net VDDA: C7.2, C8.2, FB1.1, U4.8 (VDDA)
- new net VREFN: C10.1, C11.1, FB4.1, U4.12 (VREFN)
- new net VREFP: C10.2, C11.2, FB3.1, U4.10 (VREFP)
- new net VSSA: C7.1, C8.1, FB2.1, U4.9 (VSSA)
- no-connect marks 32 -> 35
Other:
- moved on the sheet: C14, C18, C22, C32, R3
