File: hardware/artichoke/artichoke.sch (KiCad schematic (older format))
At the start: 85 parts, among them J1 USB-DEVICE, P1 SMA-CONN, P10 ATEST1, P11 ATEST2, P12 DCLK, P13 DIO, P2 PROGRAM, P3 JTAG, P4 EXPAND, P5 1V8, P6 3V3, P7 VBUS, P8 GIO1, P9 GIO6, Q1 BC856, U1 CC2591, U3 ADF7242, U4 LPC175X, U6 IP4220CZ6, U7 TPS71219, X1 ABMM2

Commit message: Artichoke schematic mostly done
Parts:
- removed C1: 2p2, 0402, symbol C
- removed C12, C14, C2, C6: 1nF, 0402, symbol C
- removed C15, C23: 68pF, 0402, symbol C
- removed C16: 100nF, 0402, symbol C
- removed C18, C32: 2.2µF, 0603, symbol C
- removed C19, C21: 27pF, 0603, symbol C
- removed C22: 1µF, 0603, symbol C
- removed C29: 220pF, 0603, symbol C
- removed C3: 1pF, 0402, symbol C
- removed C31: 100pF, 0603, symbol C
- removed C35: 10nF, 0603, symbol C
- removed C36: 15pF, 0603, symbol C
- removed C4: 18pF, 0402, symbol C
- removed C5: 6p8, 0402, symbol C
- removed C9: 10pF, 0402, symbol C
- removed D1: 1V8LED, 0603D, symbol LED
- removed FB5: FILTER, 0603, symbol FILTER
- removed L1: 3nH, 0402, symbol INDUCTOR
- removed L2: 2n2, 0402, symbol INDUCTOR
- removed L3: DNP, 0402gap, symbol INDUCTOR
- removed P10: ATEST1, testpad-50mil, symbol CONN_1
- removed P11: ATEST2, testpad-50mil, symbol CONN_1
- removed P8: GIO1, testpad-50mil, symbol CONN_1
- removed P9: GIO6, testpad-50mil, symbol CONN_1
- removed R1: 4k3, 0402, symbol R
- removed R17, R3: 10k, 0603, symbol R
- removed R18: 49.9k, 0603, symbol R
- removed R19: 30.1k, 0603, symbol R
- removed R2: 43k, 0402, symbol R
- removed R4: 330, 0603, symbol R
- removed U1: CC2591, VQFN16, symbol CC2591
- removed U7: TPS71219, S-PVSON-N10, symbol TPS712XX
- removed X1: ABMM2, ABMM2, symbol CRYSTAL
- added C?: 1µF, 0603, symbol C
- added C?: 2.2µF, 0603, symbol C
- added C?: 100nF, 0603, symbol C
- added C? (x2): 15pF, 0603, symbol C
- added C? (x2): 10nF, symbol C
- added C? (x8): 27pF, symbol C
- added C? (x2): 1pF, 0402, symbol C
- added C? (x4): 220nF, symbol C
- added C? (x2): 18pF, symbol C
- added C? (x2): 100nF, symbol C
- added L?: 9n5, symbol INDUCTOR
- added L? (x2): 2n7, symbol INDUCTOR
- added P?: ATB, symbol CONN_6
- added R?: 27k, symbol R
- added R?: 10k, 0603, symbol R
- added U?: SI9183-A, symbol SI9183-A
- added X?: NX3225SA, ABMM2, symbol CRYSTAL
- added X?: NX8045GB, ABMM2, symbol CRYSTAL
Connections:
- net labels removed: EN, GIO1, GIO6, HGM
- wire segments 306 -> 266
Other:
- note removed: "transmission\nline inductor"

Commit message: artichoke part selection
Parts:
- removed C?: 15pF, 0603, symbol C
- removed C?: 10nF, symbol C
- removed C? (x7): 27pF, symbol C
- removed C? (x3): 220nF, symbol C
- removed C?: 18pF, symbol C
- removed C?: 100nF, symbol C
- removed L?: 2n7, symbol INDUCTOR
- added C?: 18pF, symbol C
- added C?: 18pF, 0603, symbol C
- added C?: 10nF, symbol C
- added C? (x7): 27pF, symbol C
- added C? (x2): 100nF, symbol C
- added C? (x2): 220nF, symbol C
- added L?: 2n7, symbol INDUCTOR
- added P11: DCLK, testpad-50mil, symbol CONN_1
- C?: value 15pF -> 18pF; Field1 (none) -> TDK; Field2 (none) -> C1608C0G1H180JT; Field3 (none) -> Multilayer Ceramic Capacitors (MLCC) - SMD/SMT 0603 18pF 50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
- C?: Field1 (none) -> Murata; Field2 (none) -> GRM155R71H103KA88D; Field3 (none) -> CAP CER 10000PF 50V X7R 0402
- C?: Field1 (none) -> TDK; Field2 (none) -> C1005C0G1H270JT; Field3 (none) -> Multilayer Ceramic Capacitors (MLCC) - SMD/SMT 0402 27pF 50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
- C?: Field1 (none) -> TDK; Field2 (none) -> C1005X5R1C224K; Field3 (none) -> CAP CER .22UF 16V X5R 0402
- C?: Field1 (none) -> Murata; Field2 (none) -> GRM1555C1H180JZ01D; Field3 (none) -> Multilayer Ceramic Capacitors (MLCC) - SMD/SMT 0402 18pF 50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
- C?: Field1 (none) -> Murata; Field2 (none) -> GRM155R71C104KA88D; Field3 (none) -> Multilayer Ceramic Capacitors (MLCC) - SMD/SMT 0402 0.1uF 1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
- L?: Field1 (none) -> Wurth; Field2 (none) -> 744765095A; Field3 (none) -> INDUCTOR 9.5NH .68A WW 0402
- L?: Field1 (none) -> Murata; Field2 (none) -> LQW15AN2N7C00D; Field3 (none) -> RF Inductors 2.7 NH +-.2NH
- R?: Field1 (none) -> Panasonic; Field2 (none) -> ERJ-2RKF2702X; Field3 (none) -> Thick Film Resistors - SMD Thick Film Chip Res 0402 1/16W 1%
- X?: value NX8045GB -> ABM8G; footprint ABMM2 -> (none); Field1 NDK -> Abracon; Field2 NX8045GB-12.000000MHZ -> ABM8G-16.000MHZ-B4Y-T; Field3 CRYSTAL 12.000000 MHZ 8PF SMD -> CRYSTAL 16.000 MHZ 10 PF SMD
Connections:
- net DCLK is gone; now on net DT: P12.1
- net DIO is gone; now on net DR: P13.1
- net 3V3D: now also C?.2
- net GND: now also C?.1, C?.1, C?.1, C?.1, C?.1, C?.2, C?.2, C?.2, C?.2, C?.2, C?.2, C?.2, C?.2, L?.2
- net TRCLK: now also P11.1
- net at U4.20 (XTAL2), X?.2: now also C?.2
- net at C?.2, U3.1 (VDD_RF1): now also C?.2
- net at U3.10 (VCOGUARD), U3.9 (VDD_VCO): now also C?.1, C?.1
- net at U3.11 (VDD_SYNTH): now also C?.1, C?.1
- net at U3.13 (XOSC26N), X?.2: now also C?.1
- net at U3.14 (DGUARD), U3.15 (VDD_DIG2): now also C?.1, C?.1
- net at U3.27 (VDD_DIG): now also C?.2, C?.2
- net at U3.7 (RFIO2N): now also C?.2
- net at U3.8 (VDD_RF3): now also C?.1
- net at C?.1, L?.1, L?.2: now also C?.1
- net at C?.1, C?.2, L?.1: now also L?.1

Commit message: artichoke: fixed some erc errors, removed ADC section
Parts:
- removed C10, C7: 10nF, 0603, symbol C
- removed C11, C8: 1µF, 0603, symbol C
- removed FB1, FB2, FB3, FB4: FILTER, 0603bridged, symbol FILTER
- removed P5: 1V8, testpad-50mil, symbol CONN_1
- removed U3: ADF7242, symbol ADF7242
- added U2: ADF7242, symbol ADF7242
- gave numbers to parts that had none: 34
Connections:
- net 3V3 is gone; now on net 3V3D: P6.1
- net VDDA is gone; now on net 3V3D: U4.8 (VDDA)
- net VREFN is gone; now on net GND: U4.12 (VREFN)
- net VREFP is gone; now on net 3V3D: U4.10 (VREFP)
- net VSSA is gone; now on net GND: U4.9 (VSSA)
- net 3V3D: now also U2.30 (VDD_BAT)
- net CSN: now also U2.24 (CSN)
- net DR: now also U2.16 (DR_GP0)
- net DT: now also U2.17 (DT_GP1)
- net GND: now also C32.1, U2.0 (GND); no longer U4.19 (XTAL1), X2.1
- net IRQ1: now also U2.20 (IRQ1_GP4)
- net SCLK: now also U2.22 (SCLK)
- net SI: now also U2.23 (SI)
- net SO: now also U2.21 (SO)
- net TRCLK: now also U2.19 (TRCLK_CKO_GP3)
- net TRFS: now also U2.18 (IRQ_TRFS_GP2)
- net at C5.2, C6.2: now also U2.1 (VDD_RF1)
- net at C17.1, C18.1: now also U2.10 (VCOGUARD), U2.9 (VDD_VCO)
- net at C19.1, C20.1: now also U2.11 (VDD_SYNTH)
- net at C23.1, X1.1: now also U2.12 (XOSC26P)
- net at C24.1, X1.2: now also U2.13 (XOSC26N)
- net at C21.1, C22.1: now also U2.14 (DGUARD), U2.15 (VDD_DIG2)
- net at R2.1: now also U2.2 (RBIAS)
- net at P8.6: now also U2.25 (TXEN_GP5)
- net at P8.5: now also U2.26 (RXEN_GP6)
- net at C3.2, C4.2: now also U2.27 (VDD_DIG)
- net at P8.4: now also U2.28 (XOSC32KP_GP7_ATB1)
- net at P8.3: now also U2.29 (XOSC32KN_ATB2)
- net at C9.1: now also U2.3 (VDD_RF2)
- net at P8.2: now also U2.31 (PAVSUP_ATB3)
- net at P8.1: now also U2.32 (PABIAOP_ATB4)
- net at C13.2: now also U2.6 (RFIO2P)
- net at C14.2: now also U2.7 (RFIO2N)
- net at C15.1: now also U2.8 (VDD_RF3)
- net at C32.2: now also U4.19 (XTAL1), X2.1
- net ATEST1: no longer names the net of U4.7 (P0[25]/AD0[2]/I2SRX_SDA/TXD3)
- net ATEST2: no longer names the net of U4.6 (P0[26]/AD0[3]/AOUT/RXD3)
- no-connect marks 32 -> 34
Other:
- note removed: "optional ADC section"

Commit message: artichoke: assigned modules, 4 pin crystal symbol
Parts:
- P11: value DCLK -> TRCLK
- P12: value DCLK -> DT
- P13: value DIO -> DR
- P6: value 3V3 -> 3V3D
- X1, X2: symbol CRYSTAL -> XTAL4PIN
Connections:
- wire segments 257 -> 261
Changed lines of the file:
@@
-EESchema Schematic File Version 2  date Sun 10 Jul 2011 03:28:42 PM MDT
+EESchema Schematic File Version 2  date Sun 10 Jul 2011 04:05:27 PM MDT
 LIBS:ubertooth-symbols
 LIBS:power
@@
 $EndDescr
 Wire Wire Line
+	13000 9100 13000 9200
+Wire Wire Line
+	6200 5700 6200 5800
+Wire Wire Line
 	12800 9400 12800 9500
 Wire Wire Line
@@
 Wire Wire Line
 	12800 9000 12800 8450
+Wire Wire Line
+	6000 5800 6000 5700
+Wire Wire Line
+	13200 9200 13200 9100
+$Comp
+L GND #PWR?
+U 1 1 4E1A2210
+P 13200 9200
+F 0 "#PWR?" H 13200 9200 30  0001 C CNN
+F 1 "GND" H 13200 9130 30  0001 C CNN
+	1    13200 9200
+	1    0    0    -1
+$EndComp
+$Comp
+L GND #PWR?
+U 1 1 4E1A220D
+P 13000 9200
+F 0 "#PWR?" H 13000 9200 30  0001 C CNN
+F 1 "GND" H 13000 9130 30  0001 C CNN
+	1    13000 9200
+	1    0    0    -1
+$EndComp
+$Comp
+L GND #PWR?
+U 1 1 4E1A21F4
+P 6200 5800
+F 0 "#PWR?" H 6200 5800 30  0001 C CNN
+F 1 "GND" H 6200 5730 30  0001 C CNN
+	1    6200 5800
+	1    0    0    -1
+$EndComp
+$Comp
+L GND #PWR?
+U 1 1 4E1A21F2
+P 6000 5800
+F 0 "#PWR?" H 6000 5800 30  0001 C CNN
+F 1 "GND" H 6000 5730 30  0001 C CNN
+	1    6000 5800
+	1    0    0    -1
+$EndComp
 $Comp
 L 3V3D #PWR01
@@
 P 1200 7150
 F 0 "P11" H 1280 7150 40  0000 L CNN
-F 1 "DCLK" H 1200 7205 30  0001 C CNN
+F 1 "TRCLK" H 1200 7205 30  0001 C CNN
 F 2 "testpad-50mil" H 1200 7150 60  0001 C CNN
 F 4 "DNP" H 1200 7150 60  0001 C CNN "Field3"
@@
 F 6 "Multilayer Ceramic Capacitors (MLCC) - SMD/SMT 0603 18pF 50volts C0G 5%" H 13400 9200 60  0001 C CNN "Field3"
 	1    13400 9200
-	-1   0    0    1
+	1    0    0    -1
 $EndComp
 $Comp
@@
 F 6 "Multilayer Ceramic Capacitors (MLCC) - SMD/SMT 0402 18pF 50volts C0G 5%" H 5800 5800 60  0001 C CNN "Field3"
 	1    5800 5800
-	1    0    0    -1
+	-1   0    0    1
 $EndComp
 $Comp
@@
 $EndComp
 $Comp
-L CRYSTAL X2
+L XTAL4PIN X2
 U 1 1 4DFFDA24
 P 13100 8800
@@
 $EndComp
 $Comp
-L CRYSTAL X1
+L XTAL4PIN X1
 U 1 1 4DFFDA21
 P 6100 5400
@@
 P 1200 7550
 F 0 "P13" H 1280 7550 40  0000 L CNN
-F 1 "DIO" H 1200 7605 30  0001 C CNN
+F 1 "DR" H 1200 7605 30  0001 C CNN
 F 2 "testpad-50mil" H 1200 7550 60  0001 C CNN
 F 4 "DNP" H 1200 7550 60  0001 C CNN "Field3"
@@
 P 1200 7350
 F 0 "P12" H 1280 7350 40  0000 L CNN
-F 1 "DCLK" H 1200 7405 30  0001 C CNN
+F 1 "DT" H 1200 7405 30  0001 C CNN
 F 2 "testpad-50mil" H 1200 7350 60  0001 C CNN
 F 4 "DNP" H 1200 7350 60  0001 C CNN "Field3"
@@
 P 1200 6150
 F 0 "P6" H 1280 6150 40  0000 L CNN
-F 1 "3V3" H 1200 6205 30  0001 C CNN
+F 1 "3V3D" H 1200 6205 30  0001 C CNN
 F 2 "testpad-50mil" H 1200 6150 60  0001 C CNN
 F 4 "DNP" H 1200 6150 60  0001 C CNN "Field3"
