File: hardware/artichoke/artichoke.sch (KiCad schematic (older format))
At the start: 71 parts, among them J1 USB-DEVICE, P1 SMA-CONN, P11 TRCLK, P12 DT, P13 DR, P2 PROGRAM, P3 JTAG, P4 EXPAND, P6 3V3D, P7 VBUS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

Commit message: artichoke layout
Connections:
- wire segments 261 -> 254
Other:
- moved on the sheet: C28
