File: hardware/dandelion/dandelion.sch (KiCad schematic (older format))
At the start: 105 parts, among them J1 PCB antenna, J2 USB-MICRO-B, P1 DIGITAL, P10 GIO6, P11 DCLK, P12 DIO, P13 PCB JUMPER, P14 E8A, P15 R8C PROGRAM, P16 R8C EXPAND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

Commit message: adjusted C9 and C10 values
Parts:
- C10, C9: value 27pF -> 20pF; Field2 C1608C0G1H270J -> C1608C0G1H200J; Field3 Multilayer Ceramic Capacitors (MLCC) - SMD/SMT 0603 27pF 50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 -> Multilayer Ceramic Capacitors (MLCC) - SMD/SMT 0603 20pF 50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
Changed lines of the file:
@@
-EESchema Schematic File Version 2  date Sun 04 Sep 2011 11:04:05 PM MDT
+EESchema Schematic File Version 2  date Tue 20 Sep 2011 08:05:10 PM MDT
 LIBS:ubertooth-symbols
 LIBS:power
@@
 Sheet 1 1
 Title "Dandelion"
-Date "5 sep 2011"
+Date "21 sep 2011"
 Rev "$Rev$"
 Comp "Copyright 2010, 2011 Michael Ossmann"
@@
 P 4250 1300
 F 0 "C10" H 4300 1400 50  0000 L CNN
-F 1 "27pF" H 4300 1200 50  0000 L CNN
+F 1 "20pF" H 4300 1200 50  0000 L CNN
 F 2 "0603" H 4250 1300 60  0001 C CNN
 F 4 "TDK" H 4250 1300 60  0001 C CNN "Field1"
-F 5 "C1608C0G1H270J" H 4250 1300 60  0001 C CNN "Field2"
-F 6 "Multilayer Ceramic Capacitors (MLCC) - SMD/SMT 0603 27pF 50volts C0G 5%" H 4250 1300 60  0001 C CNN "Field3"
+F 5 "C1608C0G1H200J" H 4250 1300 60  0001 C CNN "Field2"
+F 6 "Multilayer Ceramic Capacitors (MLCC) - SMD/SMT 0603 20pF 50volts C0G 5%" H 4250 1300 60  0001 C CNN "Field3"
 	1    4250 1300
 	-1   0    0    1
@@
 P 3650 1300
 F 0 "C9" H 3700 1400 50  0000 L CNN
-F 1 "27pF" H 3700 1200 50  0000 L CNN
+F 1 "20pF" H 3700 1200 50  0000 L CNN
 F 2 "0603" H 3650 1300 60  0001 C CNN
 F 4 "TDK" H 3650 1300 60  0001 C CNN "Field1"
-F 5 "C1608C0G1H270J" H 3650 1300 60  0001 C CNN "Field2"
-F 6 "Multilayer Ceramic Capacitors (MLCC) - SMD/SMT 0603 27pF 50volts C0G 5%" H 3650 1300 60  0001 C CNN "Field3"
+F 5 "C1608C0G1H200J" H 3650 1300 60  0001 C CNN "Field2"
+F 6 "Multilayer Ceramic Capacitors (MLCC) - SMD/SMT 0603 20pF 50volts C0G 5%" H 3650 1300 60  0001 C CNN "Field3"
 	1    3650 1300
 	-1   0    0    1

Commit message: tc13bdge: note in schematic to omit D14 and D17 if you plan to operate on battery.
Other:
- note added: "D17 (1V8LED) and D14\n(RSTLED) are included in\nthe design as an option\nfor those who choose to\noperate exclusively on\nUSB power. Omit them\nif you plan to use a\nbattery."
- note added: "see note at D17"
Changed lines of the file:
@@
-EESchema Schematic File Version 2  date Tue 20 Sep 2011 08:05:10 PM MDT
+EESchema Schematic File Version 2  date Thu 27 Oct 2011 05:57:17 PM MDT
 LIBS:ubertooth-symbols
 LIBS:power
@@
 Sheet 1 1
 Title "Dandelion"
-Date "21 sep 2011"
+Date "27 oct 2011"
 Rev "$Rev$"
 Comp "Copyright 2010, 2011 Michael Ossmann"
@@
 Comment4 ""
 $EndDescr
+Text Notes 9250 9900 0    60   ~ 0
+see note at D17
+Text Notes 5250 7400 0    60   ~ 0
+D17 (1V8LED) and D14\n(RSTLED) are included in\nthe design as an option\nfor those who choose to\noperate exclusively on\nUSB power.  Omit them\nif you plan to use a\nbattery.
 Wire Wire Line
 	13350 800  13250 800
